File: Hardware/Magician_encoder.brd (EAGLE design)
At the start: 21.6 x 39.4 mm, 33 parts, among them Q1 MMBT2222A, Q2 MMBT2222A, U1 QRE1113, U2 QRE1113

Commit message: Put male SMT header on back
Parts:
- JP1: device SparkFun-Connectors:2X3 -> SparkFun-Connectors:2X3_SMT_POSTS
- moved JP1 2.84 mm to (10.8, 10.2), flipped to the bottom
Connections:
- net OUTA: now also JP1.2; no longer JP1.1
- net OUTB: now also JP1.1; no longer JP1.2
Routing:
- net GND: track 0.00 -> 2.79 mm, vias 0 -> 2
- net OUTB: track 17.6 -> 16.9 mm
- net OUTA: track 20.7 -> 21.2 mm
- net 5V: track 19.7 -> 19.8 mm, vias 6 -> 8
Other:
- board text added: "v11"
- board text removed: "v10"
Changed lines of the file:
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@@
 <?xml version="1.0" encoding="utf-8"?>
 <!DOCTYPE eagle SYSTEM "eagle.dtd">
-<eagle version="6.5.0">
+<eagle version="6.4">
 <drawing>
 <settings>
@@
 <setting verticaltext="up"/>
 </settings>
-<grid distance="0.05" unitdist="inch" unit="inch" style="lines" multiple="1" display="yes" altdistance="0.01" altunitdist="inch" altunit="inch"/>
+<grid distance="0.05" unitdist="inch" unit="inch" style="lines" multiple="1" display="yes" altdistance="0.005" altunitdist="inch" altunit="inch"/>
 <layers>
 <layer number="1" name="Top" color="4" fill="1" visible="yes" active="yes"/>
@@
 <layer number="19" name="Unrouted" color="6" fill="1" visible="yes" active="yes"/>
 <layer number="20" name="Dimension" color="6" fill="1" visible="yes" active="yes"/>
-<layer number="21" name="tPlace" color="6" fill="1" visible="yes" active="yes"/>
-<layer number="22" name="bPlace" color="6" fill="1" visible="yes" active="yes"/>
+<layer number="21" name="tPlace" color="16" fill="1" visible="yes" active="yes"/>
+<layer number="22" name="bPlace" color="14" fill="1" visible="yes" active="yes"/>
 <layer number="23" name="tOrigins" color="15" fill="1" visible="yes" active="yes"/>
 <layer number="24" name="bOrigins" color="15" fill="1" visible="yes" active="yes"/>
@@
 <wire x1="21.59" y1="0" x2="0" y2="0" width="0.2032" layer="20"/>
 <wire x1="0" y1="0" x2="0" y2="25.4" width="0.2032" layer="20"/>
-<text x="7.62" y="12.7" size="1.27" layer="22" font="vector" ratio="15" rot="MR0" align="center-left">OUTA</text>
-<text x="7.62" y="10.16" size="1.27" layer="22" font="vector" ratio="15" rot="MR0" align="center-left">VCC</text>
-<text x="7.62" y="7.62" size="1.27" layer="22" font="vector" ratio="15" rot="MR0" align="center-left">GND</text>
-<text x="13.97" y="7.62" size="1.27" layer="22" font="vector" ratio="15" rot="MR0" align="center-right">GND</text>
-<text x="13.97" y="10.16" size="1.27" layer="22" font="vector" ratio="15" rot="MR0" align="center-right">VCC</text>
-<text x="13.97" y="12.7" size="1.27" layer="22" font="vector" ratio="15" rot="MR0" align="center-right">OUTB</text>
+<text x="6.35" y="12.7" size="1.27" layer="22" font="vector" ratio="15" rot="MR0" align="center-left">OUTA</text>
+<text x="6.35" y="10.16" size="1.27" layer="22" font="vector" ratio="15" rot="MR0" align="center-left">VCC</text>
+<text x="6.35" y="7.62" size="1.27" layer="22" font="vector" ratio="15" rot="MR0" align="center-left">GND</text>
+<text x="15.24" y="7.62" size="1.27" layer="22" font="vector" ratio="15" rot="MR0" align="center-right">GND</text>
+<text x="15.24" y="10.16" size="1.27" layer="22" font="vector" ratio="15" rot="MR0" align="center-right">VCC</text>
+<text x="15.24" y="12.7" size="1.27" layer="22" font="vector" ratio="15" rot="MR0" align="center-right">OUTB</text>
 <text x="10.795" y="27.432" size="1.778" layer="22" font="vector" ratio="15" rot="MR0" align="center">Magician
 Chassis
@@
 <wire x1="19.05" y1="26.67" x2="20.32" y2="26.67" width="0.2032" layer="20"/>
 <wire x1="20.32" y1="26.67" x2="21.59" y2="25.4" width="0.2032" layer="20"/>
-<text x="7.62" y="36.83" size="1.778" layer="16" font="vector" ratio="15" rot="MR0">v10</text>
+<text x="7.62" y="36.83" size="1.778" layer="16" font="vector" ratio="15" rot="MR0">v11</text>
 </plain>
 <attributes>
@@
 <attribute name="PROD_ID" value="IC-09357" x="44.45" y="5.08" size="1.778" layer="27" display="off"/>
 </element>
-<element name="JP1" library="SparkFun-Connectors" package="2X3" value="" x="9.525" y="12.7" rot="R270"/>
+<element name="JP1" library="SparkFun-Connectors" package="2X3_SMT_POSTS" value="" x="10.795" y="10.16" rot="MR270">
+<attribute name="PROD_ID" value="CONN-11415" x="10.795" y="10.16" size="1.778" layer="28" rot="MR270" display="off"/>
+</element>
 <element name="R1" library="SparkFun-Resistors" package="0603-RES" value="100" x="5.08" y="13.97">
 <attribute name="PROD_ID" value="RES-07863" x="43.18" y="-6.35" size="1.778" layer="27" display="off"/>
@@
 <wire x1="19.558" y1="17.653" x2="19.939" y2="17.272" width="0.254" layer="1"/>
 <via x="19.939" y="17.272" extent="1-16" drill="0.508"/>
-<wire x1="7.239" y1="9.74" x2="7.962" y2="9.74" width="0.254" layer="1"/>
-<wire x1="7.962" y1="9.74" x2="8.382" y2="10.16" width="0.254" layer="1"/>
-<wire x1="8.382" y1="10.16" x2="9.525" y2="10.16" width="0.254" layer="1"/>
-<wire x1="14.351" y1="9.74" x2="13.628" y2="9.74" width="0.254" layer="1"/>
-<wire x1="13.628" y1="9.74" x2="13.208" y2="10.16" width="0.254" layer="1"/>
-<wire x1="13.208" y1="10.16" x2="12.065" y2="10.16" width="0.254" layer="1"/>
 <contactref element="U2" pad="3"/>
 <wire x1="18.31" y1="17.41" x2="19.801" y2="17.41" width="0.254" layer="1"/>
 <wire x1="19.801" y1="17.41" x2="19.939" y2="17.272" width="0.254" layer="1"/>
+<wire x1="14.351" y1="9.74" x2="15.66" y2="9.74" width="0.254" layer="1"/>
+<wire x1="15.66" y1="9.74" x2="16.51" y2="8.89" width="0.254" layer="1"/>
+<via x="16.51" y="8.89" extent="1-16" drill="0.508"/>
+<wire x1="7.239" y1="9.74" x2="5.93" y2="9.74" width="0.254" layer="1"/>
+<wire x1="5.93" y1="9.74" x2="5.08" y2="8.89" width="0.254" layer="1"/>
+<via x="5.08" y="8.89" extent="1-16" drill="0.508"/>
 </signal>
 <signal name="GND">
@@
 <contactref element="R8" pad="1"/>
 <contactref element="C4" pad="2"/>
+<wire x1="8.255" y1="7.62" x2="8.255" y2="6.223" width="0.254" layer="16"/>
+<via x="8.255" y="6.223" extent="1-16" drill="0.508"/>
+<wire x1="13.335" y1="7.62" x2="13.335" y2="6.223" width="0.254" layer="16"/>
+<via x="13.335" y="6.223" extent="1-16" drill="0.508"/>
 </signal>
 <signal name="OUTA">
-<contactref element="JP1" pad="1"/>
 <contactref element="R5" pad="1"/>
 <contactref element="Q1" pad="3"/>
@@
 <wire x1="4.445" y1="24.765" x2="9.144" y2="24.765" width="0.254" layer="16"/>
 <wire x1="9.144" y1="24.765" x2="9.525" y2="24.384" width="0.254" layer="16"/>
-<wire x1="9.525" y1="24.384" x2="9.525" y2="12.7" width="0.254" layer="16"/>
+<contactref element="JP1" pad="2"/>
+<wire x1="8.255" y1="12.7" x2="8.255" y2="13.335" width="0.254" layer="16"/>
+<wire x1="8.255" y1="13.335" x2="8.89" y2="13.97" width="0.254" layer="16"/>
+<wire x1="8.89" y1="13.97" x2="8.89" y2="15.113" width="0.254" layer="16"/>
+<wire x1="8.89" y1="15.113" x2="9.525" y2="15.748" width="0.254" layer="16"/>
+<wire x1="9.525" y1="15.748" x2="9.525" y2="24.384" width="0.254" layer="16"/>
 </signal>
 <signal name="N$5">
@@
 </signal>
 <signal name="OUTB">
-<contactref element="JP1" pad="2"/>
 <contactref element="R11" pad="1"/>
 <contactref element="Q2" pad="3"/>
@@
 <via x="15.24" y="24.892" extent="1-16" drill="0.508"/>
 <wire x1="15.24" y1="24.892" x2="15.24" y2="15.24" width="0.254" layer="16"/>
-<wire x1="15.24" y1="15.24" x2="12.7" y2="12.7" width="0.254" layer="16"/>
-<wire x1="12.7" y1="12.7" x2="12.065" y2="12.7" width="0.254" layer="16"/>
+<contactref element="JP1" pad="1"/>
+<wire x1="15.24" y1="15.24" x2="13.97" y2="13.97" width="0.254" layer="16"/>
+<wire x1="13.97" y1="13.97" x2="13.589" y2="13.97" width="0.254" layer="16"/>
+<wire x1="13.589" y1="13.97" x2="13.335" y2="13.716" width="0.254" layer="16"/>
+<wire x1="13.335" y1="13.716" x2="13.335" y2="12.7" width="0.254" layer="16"/>
 </signal>
 <signal name="N$10">
