File: Hardware/Magician_encoder.sch (EAGLE design)
At the start: 31 parts, among them Q1 MMBT2222A, Q2 MMBT2222A, U1 QRE1113, U2 QRE1113

Commit message: Production ready v10
Fiducial addition and panel creation
Parts:
- added FID1, FID2: FIDUCIALUFIDUCIAL, SparkFun-Aesthetics:FIDUCIALUFIDUCIAL
Changed lines of the file:
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@@
 <?xml version="1.0" encoding="utf-8"?>
 <!DOCTYPE eagle SYSTEM "eagle.dtd">
-<eagle version="6.4">
+<eagle version="6.5.0">
 <drawing>
 <settings>
@@
 <part name="C4" library="SparkFun-Capacitors" deviceset="0.1UF-25V(+80/-20%)(0603)" device="" value="0.1uF"/>
 <part name="R8" library="SparkFun-Resistors" deviceset="10KOHM1/10W1%(0603)" device="0603" value="10K"/>
+<part name="FID1" library="SparkFun-Aesthetics" deviceset="FIDUCIAL" device="UFIDUCIAL"/>
+<part name="FID2" library="SparkFun-Aesthetics" deviceset="FIDUCIAL" device="UFIDUCIAL"/>
 </parts>
 <sheets>
@@
 <instance part="C4" gate="G$1" x="162.56" y="114.3"/>
 <instance part="R8" gate="G$1" x="154.94" y="114.3" rot="R90"/>
+<instance part="FID1" gate="G$1" x="238.76" y="30.48"/>
+<instance part="FID2" gate="G$1" x="238.76" y="25.4"/>
 </instances>
 <busses>
